Commit message: GP2: migrate to 24 DOF (assets, env, AMP motion/loader updates)

File: legged_lab/assets/gp2_v2/urdf/gp2.urdf (robot description, URDF)
Before this commit: robot gp2, 24 links, 23 joints
Links:
- removed link base_link
- removed link imu_link
- added link imu_in_pelvis
- added link imu_in_torso
- added link left_elbow_yaw_link, mass 0.0001; visual cylinder length=0.14 radius=0.03
- added link pelvis, mass 0.987; collision mesh filename=meshes/base_link.STL; visual mesh filename=meshes/base_link.STL
- added link right_elbow_yaw_link, mass 0.0001; visual cylinder length=0.14 radius=0.03
- link left_ankle_pitch_link: geometry collision mesh filename=meshes/L_ankle_pitch_link.STL; visual mesh filename=meshes/L_ankle_pitch_link.STL
- link left_ankle_roll_link: geometry collision sphere radius=0.005; collision sphere radius=0.005
- link left_elbow_link: geometry collision mesh filename=meshes/L_elbow_link.STL; visual mesh filename=meshes/L_elbow_link.STL
- link left_hip_pitch_link: geometry collision mesh filename=meshes/L_hip_pitch_link.STL; visual mesh filename=meshes/L_hip_pitch_link.STL
- link left_hip_roll_link: geometry collision mesh filename=meshes/L_hip_roll_link.STL; visual mesh filename=meshes/L_hip_roll_link.STL
- link left_hip_yaw_link: geometry collision mesh filename=meshes/L_hip_yaw_link.STL; visual mesh filename=meshes/L_hip_yaw_link.STL
- link left_knee_link: geometry collision mesh filename=meshes/L_knee_link.STL; visual mesh filename=meshes/L_knee_link.STL
- link left_shoulder_pitch_link: geometry collision mesh filename=meshes/L_shoulder_pitch_link.STL; visual mesh filename=meshes/L_shoulder_pitch_link.STL
- link left_shoulder_roll_link: geometry collision mesh filename=meshes/L_shoulder_roll_link.STL; visual mesh filename=meshes/L_shoulder_roll_link.STL
- link left_shoulder_yaw_link: geometry collision mesh filename=meshes/L_shoulder_yaw_link.STL; visual mesh filename=meshes/L_shoulder_yaw_link.STL
- link right_ankle_pitch_link: geometry collision mesh filename=meshes/R_ankle_pitch_link.STL; visual mesh filename=meshes/R_ankle_pitch_link.STL
- link right_ankle_roll_link: geometry collision sphere radius=0.005; collision sphere radius=0.005
- link right_elbow_link: geometry collision mesh filename=meshes/R_elbow_link.STL; visual mesh filename=meshes/R_elbow_link.STL
- link right_hip_pitch_link: geometry collision mesh filename=meshes/R_hip_pitch_link.STL; visual mesh filename=meshes/R_hip_pitch_link.STL
- link right_hip_roll_link: geometry collision mesh filename=meshes/R_hip_roll_link.STL; visual mesh filename=meshes/R_hip_roll_link.STL
- link right_hip_yaw_link: geometry collision mesh filename=meshes/R_hip_yaw_link.STL; visual mesh filename=meshes/R_hip_yaw_link.STL
- link right_knee_link: geometry collision mesh filename=meshes/R_knee_link.STL; visual mesh filename=meshes/R_knee_link.STL
- link right_shoulder_pitch_link: geometry collision mesh filename=meshes/R_shoulder_pitch_link.STL; visual mesh filename=meshes/R_shoulder_pitch_link.STL
- link right_shoulder_roll_link: geometry collision mesh filename=meshes/R_shoulder_roll_link.STL; visual mesh filename=meshes/R_shoulder_roll_link.STL
- link right_shoulder_yaw_link: geometry collision mesh filename=meshes/R_shoulder_yaw_link.STL; visual mesh filename=meshes/R_shoulder_yaw_link.STL
- link torso_link: geometry collision mesh filename=meshes/waist_roll_link.STL; visual mesh filename=meshes/waist_roll_link.STL
- link waist_yaw_link: geometry collision mesh filename=meshes/waist_yaw_link.STL; visual mesh filename=meshes/waist_yaw_link.STL
Joints:
- removed joint imu_joint
- added joint imu_in_pelvis_joint: type fixed, parent pelvis, child imu_in_pelvis, origin xyz=0 0 -0.0057 rpy=0 0 0
- added joint imu_in_torso_joint: type fixed, parent torso_link, child imu_in_torso, origin xyz=-0.04 0 0.1835 rpy=0 0 0
- added joint left_elbow_yaw_joint: type revolute, parent left_elbow_link, child left_elbow_yaw_link, origin xyz=-0.02 -0.035 0 rpy=1.5707963267949 -1.5708 0, axis 1 0 0, limit lower=-1.5708 upper=1.5708 effort=25 velocity=37
- added joint right_elbow_yaw_joint: type revolute, parent right_elbow_link, child right_elbow_yaw_link, origin xyz=-0.02 0.035 0 rpy=1.5707963267949 -1.5708 0, axis 1 0 0, limit lower=-1.5708 upper=1.5708 effort=25 velocity=37
- joint left_ankle_pitch_joint: limit lower=-0.87267 upper=0.5236 effort=50 velocity=37 -> lower=-0.349 upper=0.349 effort=50 velocity=37
- joint left_elbow_joint: origin xyz=0.0200000000000853 0.0339999999999863 -0.0704999999999717 rpy=0 0 0 -> xyz=0.0200000000000853 0.0339999999999863 -0.0704999999999717 rpy=0 -1.5707963267948966 0; type fixed -> revolute
- joint left_hip_pitch_joint: parent base_link -> pelvis
- joint left_shoulder_roll_joint: type fixed -> revolute
- joint left_shoulder_yaw_joint: type fixed -> revolute
- joint right_ankle_pitch_joint: limit lower=-0.87267 upper=0.5236 effort=50 velocity=37 -> lower=-0.349 upper=0.349 effort=50 velocity=37
- joint right_elbow_joint: origin xyz=0.0200000000001179 -0.0340000000000086 -0.0704999999999668 rpy=0 0 0 -> xyz=0.0200000000001179 -0.0340000000000086 -0.0704999999999668 rpy=0 -1.5707963267948966 0; type fixed -> revolute
- joint right_hip_pitch_joint: parent base_link -> pelvis
- joint right_shoulder_roll_joint: type fixed -> revolute
- joint right_shoulder_yaw_joint: type fixed -> revolute
- joint waist_roll_joint: type fixed -> revolute
- joint waist_yaw_joint: parent base_link -> pelvis; type fixed -> revolute

Commit message: trim down to 21 dof, add penalty for upper bodies movement, switch motion files, lower kps

File: legged_lab/assets/gp2_v2/urdf/gp2.urdf (robot description, URDF)
Before this commit: robot GP02, 27 links, 26 joints
Joints:
- joint left_elbow_yaw_joint: axis 1 0 0 -> (none); limit lower=-1.5708 upper=1.5708 effort=25 velocity=37 -> (none); type revolute -> fixed
- joint right_elbow_yaw_joint: axis 1 0 0 -> (none); limit lower=-1.5708 upper=1.5708 effort=25 velocity=37 -> (none); type revolute -> fixed
- joint waist_roll_joint: axis 1 0 0 -> (none); limit lower=-0.17 upper=0.17 effort=50 velocity=37 -> (none); type revolute -> fixed

Commit message: decrease range for waist_yaw, new motion

File: legged_lab/assets/gp2_v2/urdf/gp2.urdf (robot description, URDF)
Before this commit: robot GP02, 27 links, 26 joints
Joints:
- joint waist_yaw_joint: limit lower=-2.79 upper=2.79 effort=88 velocity=32 -> lower=-0.25 upper=0.25 effort=88 velocity=32
