Commit message: almost ready to run except setMass error

File: legged_lab/assets/gp2_v2/urdf/gp02-v3.urdf (robot description, URDF)
Before this commit: robot GP02-V3, 25 links, 24 joints
Links:
- added link imu_in_pelvis; visual sphere radius=0.005
- added link imu_in_torso; visual sphere radius=0.005
Joints:
- added joint imu_in_pelvis_joint: type fixed, parent pelvis, child imu_in_pelvis, origin xyz=0 0 0 rpy=0 0 0
- added joint imu_in_torso_joint: type fixed, parent torso_link, child imu_in_torso, origin xyz=0.07 0 0.04 rpy=0 0 0
- joint left_shoulder_pitch_joint: origin xyz=0.11844 0.001 0.241 rpy=0 0 -1.5708 -> xyz=-0.001 0.11844 0.241 rpy=0 0 0
- joint right_shoulder_pitch_joint: origin xyz=-0.11844 0.001 0.241 rpy=0 0 -1.5708 -> xyz=-0.001 -0.11844 0.241 rpy=0 0 0
- joint waist_roll_joint: axis 0 1 0 -> 1 0 0; origin xyz=0.001 0 0.0522 rpy=0 0 1.5708 -> xyz=0.001 0 0.0522 rpy=0 0 0
