Commit message: x2 step up effort

File: legged_lab/assets/X2_URDF-v1.3.0/x2_hand.urdf (robot description, URDF)
Before this commit: robot x2_t2.5, 35 links, 34 joints
Joints:
- joint head_pitch_joint: type revolute -> fixed
- joint head_yaw_joint: type revolute -> fixed
- joint left_wrist_yaw_joint: type revolute -> fixed
- joint right_wrist_yaw_joint: type revolute -> fixed
- joint waist_pitch_joint: type revolute -> fixed
- joint waist_roll_joint: type revolute -> fixed
